File: DRC-PumpDriver2026.kicad_pcb (KiCad board)
At the start: 2 copper layers, 80 x 60 mm, 89 parts, among them J1 STLINK, J10 Vin_PWR, J2 CAN, J3 CAN, J4 PUMP1, J5 PUMP2, J6 PUMP3, J7 PUMP4, J8 PUMP5, J9 PUMP6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

Commit message: シルクスクリーンと被らないようにビアを調整
Routing:
- net GNDPWR: vias 47 -> 44
Changed lines of the file:
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@@
-	)
-	(via
-		(at 120.65 83.18)
-		(size 1.3)
-		(drill 1)
-		(layers "F.Cu" "B.Cu")
-		(free yes)
-		(net 6)
 	)
 	(via
@@
 	(via
 		(at 190.5 95.88)
-		(size 1.3)
-		(drill 1)
-		(layers "F.Cu" "B.Cu")
-		(free yes)
-		(net 6)
-	)
-	(via
-		(at 120.65 80.64)
 		(size 1.3)
 		(drill 1)
@@
 		(size 1.3)
 		(drill 1)
-		(layers "F.Cu" "B.Cu")
-		(free yes)
-		(net 6)
-	)
-	(via
-		(at 120.65 78.1)
-		(size 1.3)
-		(drill 1)
