File: TJA1441.kicad_sch (KiCad schematic)
At the start: 5 parts

Commit message: DCDCを外して、電源入力に変更、v0.0.2
Parts:
- removed JP1: TR, Jumper:SolderJumper-2_P1.3mm_Open_RoundedPad1.0x1.5mm, symbol Jumper:SolderJumper_2_Open
- added SW3: SS-12D00G3, lib:SS-12D00G3, symbol lib:SS-12D00G3
- renumbered C21 to C7, C22 to C8, R25 to R17
Connections:
- net CAN_H: now also SW3.2 (B)
- net CAN_L: now also SW3.3 (C)
- net at R17.1: now also SW3.1 (A)
Other:
- moved on the sheet: R17
Changed lines of the file:
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@@
 	)
 	(junction
-		(at 120.65 74.93)
+		(at 125.73 77.47)
 		(diameter 0)
 		(color 0 0 0 0)
 	)
 	(junction
-		(at 120.65 59.69)
+		(at 123.19 57.15)
+		(diameter 0)
+		(color 0 0 0 0)
+	)
+	(junction
+		(at 120.65 77.47)
 		(diameter 0)
 		(color 0 0 0 0)
@@
 	(wire
 		(pts
+			(xy 120.65 77.47) (xy 125.73 77.47)
+		)
+		(stroke
+			(width 0)
+			(type default)
+		)
+	)
+	(wire
+		(pts
 			(xy 78.74 69.85) (xy 82.55 69.85)
 		)
@@
 	(wire
 		(pts
-			(xy 120.65 59.69) (xy 124.46 59.69)
+			(xy 123.19 57.15) (xy 133.35 57.15)
 		)
 		(stroke
@@
 	(wire
 		(pts
-			(xy 118.11 74.93) (xy 120.65 74.93)
+			(xy 118.11 77.47) (xy 120.65 77.47)
 		)
 		(stroke
@@
 	(wire
 		(pts
-			(xy 118.11 71.12) (xy 118.11 74.93)
+			(xy 118.11 71.12) (xy 118.11 77.47)
 		)
 		(stroke
@@
 	(wire
 		(pts
-			(xy 120.65 73.66) (xy 120.65 74.93)
+			(xy 125.73 76.2) (xy 125.73 77.47)
 		)
 		(stroke
@@
 	(wire
 		(pts
-			(xy 118.11 59.69) (xy 118.11 63.5)
-		)
-		(stroke
-			(width 0)
-			(type default)
-		)
-	)
-	(wire
-		(pts
-			(xy 118.11 59.69) (xy 120.65 59.69)
+			(xy 118.11 57.15) (xy 118.11 63.5)
+		)
+		(stroke
+			(width 0)
+			(type default)
+		)
+	)
+	(wire
+		(pts
+			(xy 118.11 57.15) (xy 123.19 57.15)
 		)
 		(stroke
@@
 	(wire
 		(pts
-			(xy 120.65 59.69) (xy 120.65 60.96)
+			(xy 123.19 57.15) (xy 123.19 60.96)
 		)
 		(stroke
@@
 	(wire
 		(pts
-			(xy 120.65 74.93) (xy 124.46 74.93)
+			(xy 120.65 71.12) (xy 120.65 77.47)
+		)
+		(stroke
+			(width 0)
+			(type default)
+		)
+	)
+	(wire
+		(pts
+			(xy 125.73 77.47) (xy 133.35 77.47)
 		)
 		(stroke
@@
 	(hierarchical_label "CAN_L"
 		(shape bidirectional)
-		(at 124.46 74.93 0)
+		(at 133.35 77.47 0)
 		(effects
 			(font
@@
 	(hierarchical_label "CAN_H"
 		(shape bidirectional)
-		(at 124.46 59.69 0)
+		(at 133.35 57.15 0)
 		(effects
 			(font
@@
 		(on_board yes)
 		(dnp no)
-		(property "Reference" "#PWR062"
+		(property "Reference" "#PWR038"
 			(at 78.74 77.47 0)
 			(effects
@@
 			(project "DRC-PumpDriver2026"
 				(path "/cf42be67-fab3-494c-b2b5-38aff4068810/3a4a56d4-04c8-4cdb-9269-7809d127a6ab"
-					(reference "#PWR062")
-					(unit 1)
-				)
-			)
-		)
-	)
-	(symbol
-		(lib_id "Jumper:SolderJumper_2_Open")
-		(at 120.65 64.77 270)
-		(unit 1)
-		(exclude_from_sim no)
-		(in_bom no)
-		(on_board yes)
-		(dnp no)
-		(property "Reference" "JP1"
-			(at 121.92 63.5 90)
-			(effects
-				(font
-					(size 1.27 1.27)
-				)
-				(justify left)
-			)
-		)
-		(property "Value" "TR"
-			(at 121.92 66.04 90)
-			(effects
-				(font
-					(size 1.27 1.27)
-				)
-				(justify left)
-			)
-		)
-		(property "Footprint" "Jumper:SolderJumper-2_P1.3mm_Open_RoundedPad1.0x1.5mm"
-			(at 120.65 64.77 0)
-			(effects
-				(font
-					(size 1.27 1.27)
-				)
-				(hide yes)
-			)
-		)
-		(property "Datasheet" "~"
-			(at 120.65 64.77 0)
-			(effects
-				(font
-					(size 1.27 1.27)
-				)
-				(hide yes)
-			)
-		)
-		(property "Description" "Solder Jumper, 2-pole, open"
-			(at 120.65 64.77 0)
-			(effects
-				(font
-					(size 1.27 1.27)
-				)
-				(hide yes)
-			)
-		)
-		(pin "1"
-		)
-		(pin "2"
-		)
-		(instances
-			(project "DRC-PumpDriver2026"
-				(path "/cf42be67-fab3-494c-b2b5-38aff4068810/3a4a56d4-04c8-4cdb-9269-7809d127a6ab"
-					(reference "JP1")
+					(reference "#PWR038")
 					(unit 1)
 				)
@@
 		(on_board yes)
 		(dnp no)
-		(property "Reference" "C21"
+		(property "Reference" "C7"
 			(at 84.328 68.834 90)
 			(effects
@@
 			(project "DRC-PumpDriver2026"
 				(path "/cf42be67-fab3-494c-b2b5-38aff4068810/3a4a56d4-04c8-4cdb-9269-7809d127a6ab"
-					(reference "C21")
+					(reference "C7")
 					(unit 1)
 				)
@@
 		(on_board yes)
 		(dnp no)
-		(property "Reference" "#PWR066"
+		(property "Reference" "#PWR042"
 			(at 104.14 88.9 0)
 			(effects
@@
 			(project "DRC-PumpDriver2026"
 				(path "/cf42be67-fab3-494c-b2b5-38aff4068810/3a4a56d4-04c8-4cdb-9269-7809d127a6ab"
-					(reference "#PWR066")
+					(reference "#PWR042")
 					(unit 1)
 				)
@@
 	(symbol
 		(lib_id "lib:R_Small")
-		(at 120.65 71.12 0)
+		(at 125.73 73.66 0)
 		(unit 1)
 		(exclude_from_sim no)
@@
 		(on_board yes)
 		(dnp no)
-		(property "Reference" "R25"
-			(at 121.92 69.85 0)
+		(property "Reference" "R17"
+			(at 127 72.39 0)
 			(effects
 				(font
@@
 		)
 		(property "Value" "120"
-			(at 121.92 72.39 0)
+			(at 127 74.93 0)
 			(effects
 				(font
@@
 		)
 		(property "Footprint" "Resistor_SMD:R_0603_1608Metric_Pad0.98x0.95mm_HandSolder"
-			(at 120.65 71.12 0)
+			(at 125.73 73.66 0)
 			(effects
 				(font
@@
 		)
 		(property "Datasheet" "~"
-			(at 120.65 71.12 0)
+			(at 125.73 73.66 0)
 			(effects
 				(font
@@
 		)
 		(property "Description" "Resistor, small symbol"
-			(at 120.65 71.12 0)
+			(at 125.73 73.66 0)
 			(effects
 				(font
@@
 			(project "DRC-PumpDriver2026"
 				(path "/cf42be67-fab3-494c-b2b5-38aff4068810/3a4a56d4-04c8-4cdb-9269-7809d127a6ab"
-					(reference "R25")
+					(reference "R17")
 					(unit 1)
 				)
@@
 		(on_board yes)
 		(dnp no)
-		(property "Reference" "C22"
+		(property "Reference" "C8"
 			(at 100.33 49.022 90)
 			(effects
@@
 			(project "DRC-PumpDriver2026"
 				(path "/cf42be67-fab3-494c-b2b5-38aff4068810/3a4a56d4-04c8-4cdb-9269-7809d127a6ab"
-					(reference "C22")
+					(reference "C8")
 					(unit 1)
 				)
@@
 		(on_board yes)
 		(dnp no)
-		(property "Reference" "#PWR063"
+		(property "Reference" "#PWR039"
 			(at 88.9 72.39 0)
 			(effects
@@
 			(project "DRC-PumpDriver2026"
 				(path "/cf42be67-fab3-494c-b2b5-38aff4068810/3a4a56d4-04c8-4cdb-9269-7809d127a6ab"
-					(reference "#PWR063")
+					(reference "#PWR039")
 					(unit 1)
 				)
@@
 		(on_board yes)
 		(dnp no)
-		(property "Reference" "#PWR064"
+		(property "Reference" "#PWR040"
 			(at 96.52 60.96 0)
 			(effects
@@
 			(project "DRC-PumpDriver2026"
 				(path "/cf42be67-fab3-494c-b2b5-38aff4068810/3a4a56d4-04c8-4cdb-9269-7809d127a6ab"
-					(reference "#PWR064")
+					(reference "#PWR040")
+					(unit 1)
+				)
+			)
+		)
+	)
+	(symbol
+		(lib_id "lib:SS-12D00G3")
+		(at 123.19 66.04 270)
+		(unit 1)
+		(exclude_from_sim no)
+		(in_bom yes)
+		(on_board yes)
+		(dnp no)
+		(fields_autoplaced yes)
+		(property "Reference" "SW3"
+			(at 128.27 64.7699 90)
+			(effects
+				(font
+					(size 1.27 1.27)
+				)
+				(justify left)
+			)
+		)
+		(property "Value" "SS-12D00G3"
+			(at 128.27 67.3099 90)
+			(effects
+				(font
+					(size 1.27 1.27)
+				)
+				(justify left)
+			)
+		)
+		(property "Footprint" "lib:SS-12D00G3"
+			(at 123.19 66.04 0)
+			(effects
+				(font
+					(size 1.27 1.27)
+				)
+				(hide yes)
+			)
+		)
+		(property "Datasheet" ""
+			(at 123.19 66.04 0)
+			(effects
+				(font
+					(size 1.27 1.27)
+				)
+				(hide yes)
+			)
+		)
+		(property "Description" ""
+			(at 123.19 66.04 0)
+			(effects
+				(font
+					(size 1.27 1.27)
+				)
+				(hide yes)
+			)
+		)
+		(pin "3"
+		)
+		(pin "1"
+		)
+		(pin "2"
+		)
+		(instances
+			(project "DRC-PumpDriver2026"
+				(path "/cf42be67-fab3-494c-b2b5-38aff4068810/3a4a56d4-04c8-4cdb-9269-7809d127a6ab"
+					(reference "SW3")
 					(unit 1)
 				)
@@
 		(on_board yes)
 		(dnp no)
-		(property "Reference" "#PWR065"
+		(property "Reference" "#PWR041"
 			(at 104.14 55.88 0)
 			(effects
@@
 			(project "DRC-PumpDriver2026"
 				(path "/cf42be67-fab3-494c-b2b5-38aff4068810/3a4a56d4-04c8-4cdb-9269-7809d127a6ab"
-					(reference "#PWR065")
+					(reference "#PWR041")
 					(unit 1)
 				)
